File: sweeper.sch (KiCad schematic (older format))
At the start: 16 parts, among them Q1 2N7000, U1 LM7805_TO220, U2 PIC12F675-IP, Y1 12MHz

Commit message: Update circuit.
Parts:
- added J1, J2: Conn_01x02, symbol Connector_Generic:Conn_01x02
- added J3: Jack-DC, symbol Connector:Jack-DC
Connections:
- net +12V: now also J1.1 (Pin_1), J3.1
- net GND: now also J1.2 (Pin_2), J3.2
- net at LS1.2, Q1.3 (D): now also J2.2 (Pin_2)
- net at LS1.1, R4.1: now also J2.1 (Pin_1)
Other:
- moved on the sheet: LS1
Changed lines of the file:
@@
 L Device:Speaker LS1
 U 1 1 5CD6017A
-P 7050 2800
-F 0 "LS1" H 7220 2796 50  0000 L CNN
-F 1 "Speaker" H 7220 2705 50  0000 L CNN
-F 2 "" H 7050 2600 50  0001 C CNN
-F 3 "~" H 7040 2750 50  0001 C CNN
-	1    7050 2800
+P 7250 2800
+F 0 "LS1" H 7420 2796 50  0000 L CNN
+F 1 "Speaker" H 7420 2705 50  0000 L CNN
+F 2 "" H 7250 2600 50  0001 C CNN
+F 3 "~" H 7240 2750 50  0001 C CNN
+	1    7250 2800
 	1    0    0    -1
 $EndComp
@@
 L power:+12V #PWR01
 U 1 1 5CD676BF
-P 2350 3100
-F 0 "#PWR01" H 2350 2950 50  0001 C CNN
-F 1 "+12V" H 2365 3273 50  0000 C CNN
-F 2 "" H 2350 3100 50  0001 C CNN
-F 3 "" H 2350 3100 50  0001 C CNN
-	1    2350 3100
+P 1800 2550
+F 0 "#PWR01" H 1800 2400 50  0001 C CNN
+F 1 "+12V" H 1815 2723 50  0000 C CNN
+F 2 "" H 1800 2550 50  0001 C CNN
+F 3 "" H 1800 2550 50  0001 C CNN
+	1    1800 2550
 	1    0    0    -1
 $EndComp
@@
 Wire Wire Line
 	3500 4650 3500 4450
-Wire Wire Line
-	2350 3100 2350 3250
 $Comp
 L Device:Crystal Y1
@@
 Wire Wire Line
 	2900 3250 2900 3450
-Wire Wire Line
-	6850 2900 6850 3550
 $Comp
 L Device:R R4
@@
 Wire Wire Line
 	2800 3250 2900 3250
-Wire Wire Line
-	2500 3250 2350 3250
 NoConn ~ 5900 3850
+Wire Wire Line
+	6850 3550 6850 2950
+$Comp
+L power:GND #PWR03
+U 1 1 5CDBEE27
+P 1800 3350
+F 0 "#PWR03" H 1800 3100 50  0001 C CNN
+F 1 "GND" H 1805 3177 50  0000 C CNN
+F 2 "" H 1800 3350 50  0001 C CNN
+F 3 "" H 1800 3350 50  0001 C CNN
+	1    1800 3350
+	1    0    0    -1
+$EndComp
+Wire Wire Line
+	2500 3250 2250 3250
+$Comp
+L Connector_Generic:Conn_01x02 J2
+U 1 1 5CDC1EE7
+P 6500 2800
+F 0 "J2" H 6418 3017 50  0000 C CNN
+F 1 "Conn_01x02" H 6418 2926 50  0000 C CNN
+F 2 "" H 6500 2800 50  0001 C CNN
+F 3 "~" H 6500 2800 50  0001 C CNN
+	1    6500 2800
+	-1   0    0    -1
+$EndComp
+$Comp
+L Connector_Generic:Conn_01x02 J1
+U 1 1 5CDC55FE
+P 2000 3000
+F 0 "J1" H 2080 2992 50  0000 L CNN
+F 1 "Conn_01x02" H 2080 2901 50  0000 L CNN
+F 2 "" H 2000 3000 50  0001 C CNN
+F 3 "~" H 2000 3000 50  0001 C CNN
+	1    2000 3000
+	1    0    0    -1
+$EndComp
+Wire Wire Line
+	6700 2800 6850 2800
+Connection ~ 6850 2800
+Wire Wire Line
+	6700 2900 6850 2900
+Wire Wire Line
+	6850 2900 6850 2950
+Connection ~ 6850 2950
+Wire Wire Line
+	7050 2950 7050 2900
+$Comp
+L power:+12V #PWR04
+U 1 1 5CDD6324
+P 2250 2550
+F 0 "#PWR04" H 2250 2400 50  0001 C CNN
+F 1 "+12V" H 2265 2723 50  0000 C CNN
+F 2 "" H 2250 2550 50  0001 C CNN
+F 3 "" H 2250 2550 50  0001 C CNN
+	1    2250 2550
+	1    0    0    -1
+$EndComp
+Wire Wire Line
+	2250 2550 2250 3250
+Wire Wire Line
+	1800 3100 1800 3150
+Wire Wire Line
+	1800 2550 1800 2950
+Wire Wire Line
+	6850 2950 7050 2950
+Wire Wire Line
+	6850 2800 7050 2800
+$Comp
+L Connector:Jack-DC J3
+U 1 1 5CDDC92B
+P 1350 3050
+F 0 "J3" H 1407 3375 50  0000 C CNN
+F 1 "Jack-DC" H 1407 3284 50  0000 C CNN
+F 2 "" H 1400 3010 50  0001 C CNN
+F 3 "~" H 1400 3010 50  0001 C CNN
+	1    1350 3050
+	1    0    0    -1
+$EndComp
+Wire Wire Line
+	1650 3150 1800 3150
+Connection ~ 1800 3150
+Wire Wire Line
+	1800 3150 1800 3350
+Wire Wire Line
+	1650 2950 1800 2950
+Connection ~ 1800 2950
+Wire Wire Line
+	1800 2950 1800 3000
 $EndSCHEMATC

Commit message: Update circuit.
Parts:
- R4: value 1k -> 3.9
Changed lines of the file:
@@
 EESchema Schematic File Version 4
-LIBS:sweeper-cache
-EELAYER 29 0
+EELAYER 30 0
 EELAYER END
 $Descr A4 11693 8268
@@
 P 4650 2450
 F 0 "R4" V 4550 2300 50  0000 L CNN
-F 1 "1k" V 4550 2500 50  0000 L CNN
+F 1 "3.9" V 4550 2500 50  0000 L CNN
 F 2 "" V 4580 2450 50  0001 C CNN
 F 3 "~" H 4650 2450 50  0001 C CNN
