File: sweeper.kicad_sch (KiCad schematic)
At the start: 21 parts, among them J1 Conn_01x02, J2 Conn_01x02, J3 Jack-DC, Q1 2N7000, U1 LM7805_TO220, U2 PIC12F675-IP, Y1 12MHz

Commit message: Lower frequency and sine wave filter.
Parts:
- added C7, C8: 0.01u, symbol Device:C
- added C9: 0.1u, symbol Device:C
- added R6, R7, R8: 470, symbol Device:R
- C6: value 0.1u -> 0.01u
- R5: value 470 -> 1k
Connections:
- net GND: now also C6.1, C7.1, C8.1
- net at C2.1, C3.1, R1.1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: now also R4.2
- net at C1.1, D2.1 (K), U1.1 (VI): no longer R4.2
- net at Q1.3 (D), R5.1: now also R6.2; no longer C6.1
- net at J2.1 (Pin_1), LS1.1: now also C9.1; no longer C6.2
- new net: C8.2, C9.2, R8.1
- new net: C7.2, R7.1, R8.2
- new net: C6.2, R6.1, R7.2
Other:
- note added: "Sine Wave Filter 33.8kHz"
- note added: "~10mA"
- note removed: "+"
- note removed: "-"
- moved on the sheet: C6, J2, LS1

Commit message: Renew circuit.
Parts:
- removed C7, C8: 0.01u, symbol Device:C
- removed R7, R8: 470, symbol Device:R
- R3: renamed from R5; value 1k -> 470
- renumbered C4 to C3, C5 to C4, C3 to C5, C9 to C7, D2 to D1, D1 to D2, J3 to J1, J1 to J2, J2 to J3, R4 to R2, R2 to R4, R3 to R5
Connections:
- net at C7.2: now also C6.2, R6.1
Other:
- note removed: "~10mA"
- moved on the sheet: C7
